Commit message: Correct robot urdf

File: robot_arm_description/urdf/robot_arm.urdf (robot description, URDF)
Before this commit: robot robot_arm, 6 links, 5 joints
Links:
- removed link base_link
- added link base; visual cylinder length=0.03 radius=0.04
Joints:
- joint elbow: axis 0 1 0 -> 0 -1 0
- joint shoulder_psi: parent base_link -> base
- joint wrist_theta: axis 0 -1 0 -> 0 1 0

Commit message: Add moveit config package

File: robot_arm_description/urdf/robot_arm.urdf (robot description, URDF)
Before this commit: robot robot_arm, 6 links, 5 joints
Links:
- link arm: geometry collision mesh filename=package://robot_arm_description/models/arm.stl; visual mesh filename=package://robot_arm_description/models/arm.stl
- link base: geometry collision cylinder length=0.03 radius=0.04; visual cylinder length=0.03 radius=0.04
- link fingers: geometry collision mesh filename=package://robot_arm_description/models/fingers.stl; visual mesh filename=package://robot_arm_description/models/fingers.stl
- link forearm: geometry collision mesh filename=package://robot_arm_description/models/forearm.stl; visual mesh filename=package://robot_arm_description/models/forearm.stl
- link hand: geometry collision mesh filename=package://robot_arm_description/models/hand.stl; visual mesh filename=package://robot_arm_description/models/hand.stl
- link upper_arm: geometry collision mesh filename=package://robot_arm_description/models/upper_arm.stl; visual mesh filename=package://robot_arm_description/models/upper_arm.stl

Commit message: Fix self collisions in srdf / urdf

File: robot_arm_description/urdf/robot_arm.urdf (robot description, URDF)
Before this commit: robot robot_arm, 6 links, 5 joints
Joints:
- joint wrist_theta: origin xyz=0 0 0.0912 -> xyz=0 0 0.08698

Commit message: Shift TCP to fingertips

File: robot_arm_description/urdf/robot_arm.urdf (robot description, URDF)
Before this commit: robot robot_arm, 6 links, 5 joints
Links:
- added link tcp_link
Joints:
- added joint tcp_joint: type fixed, parent fingers, child tcp_link, origin xyz=0 0 0.06, axis 0 0 1

Commit message: Add a move group for the gripper

File: robot_arm_description/urdf/robot_arm.urdf (robot description, URDF)
Before this commit: robot robot_arm, 7 links, 6 joints
Links:
- removed link fingers
- added link carpals; collision mesh filename=package://robot_arm_description/models/carpals.stl; visual mesh filename=package://robot_arm_description/models/carpals.stl
- added link left_finger; collision mesh filename=package://robot_arm_description/models/finger.stl; visual mesh filename=package://robot_arm_description/models/finger.stl
- added link right_finger; collision mesh filename=package://robot_arm_description/models/finger.stl; visual mesh filename=package://robot_arm_description/models/finger.stl
Joints:
- added joint left_knuckle: type prismatic, parent carpals, child left_finger, origin xyz=0 0 0.031, axis 0 -1 0, limit lower=0 upper=0.03 effort=1 velocity=1
- added joint right_knuckle: type prismatic, parent carpals, child right_finger, origin xyz=0 0 0.031, axis 0 1 0, limit lower=0 upper=0.03 effort=1 velocity=1, mimic joint=left_knuckle
- joint tcp_joint: parent fingers -> carpals
- joint wrist_psi: child fingers -> carpals

File: robot_arm_moveit_config/config/robot_arm.ros2_control.xacro (robot description, xacro)
@@ -5,12 +5,13 @@
         <ros2_control name="${name}" type="system">
             <hardware>
-                <!-- By default, set up controllers for simulation. This won't work on real hardware -->
                 <plugin>robot_arm_control/RobotArmPositionOnlyHardware</plugin>
                 <param name="port">/dev/serial/by-id/usb-FTDI_Toms_FTDI_Cable_A8WW0LV8-if00-port0</param>
                 <param name="baudrate">1000000</param>
+                <param name="gripper_rad_to_meters">0.026087183366811886</param>
             </hardware>
             <joint name="shoulder_psi">
                 <param name="id">16</param>
                 <param name="offset">0.0</param>
+                <param name="multiplier">1.0</param>
                 <command_interface name="position"/>
                 <state_interface name="position">
@@ -21,4 +22,5 @@
               <param name="id">17</param>
               <param name="offset">0.04601942363656919</param>
+              <param name="multiplier">1.0</param>
               <command_interface name="position"/>
                 <state_interface name="position">
@@ -29,4 +31,5 @@
                 <param name="id">18</param>
                 <param name="offset">-0.0869255779801863</param>
+                <param name="multiplier">1.0</param>
                 <command_interface name="position"/>
                 <state_interface name="position">
@@ -37,4 +40,5 @@
                 <param name="id">19</param>
                 <param name="offset">0.04090615434361711</param>
+                <param name="multiplier">1.0</param>
                 <command_interface name="position"/>
                 <state_interface name="position">
@@ -45,4 +49,5 @@
                 <param name="id">20</param>
                 <param name="offset">0.20964404101103762</param>
+                <param name="multiplier">1.0</param>
                 <command_interface name="position"/>
                 <state_interface name="position">
@@ -50,4 +55,22 @@
                 </state_interface>
             </joint>
+            <joint name="wrist_psi">
+              <param name="id">20</param>
+              <param name="offset">0.20964404101103762</param>
+              <param name="multiplier">1.0</param>
+              <command_interface name="position"/>
+              <state_interface name="position">
+                <param name="initial_value">${initial_positions['wrist_psi']}</param>
+              </state_interface>
+            </joint>
+            <joint name="left_knuckle">
+              <param name="id">21</param>
+              <param name="offset">-0.03443484</param>
+              <param name="multiplier">0.026087183366811886</param>
+              <command_interface name="position"/>
+              <state_interface name="position">
+                <param name="initial_value">${initial_positions['left_knuckle']}</param>
+              </state_interface>
+            </joint>
         </ros2_control>
     </xacro:macro>
